File: pidyou/pidyou.kicad_sch (KiCad schematic)
At the start: 20 parts, among them J1 Conn_01x02, J2 Conn_01x02, M1 RE-280RA-2865, Q1 2SK4017(Q), Q2 2SK4017(Q), Q3 2SK4017(Q), Q4 2SK4017(Q), U1 PC817

Commit message: add pidyou
Parts:
- added C2: 0.1 uF, symbol Device:C
- added D1: OSB5YU3Z74A, symbol Device:LED
- added F1: MF-R090, symbol Device:Polyfuse
- added J10, J11, J12, J4, J5, J8: Conn_01x02, symbol Connector_Generic:Conn_01x02
- added J3, J7, J9: Conn_01x04, symbol Connector_Generic:Conn_01x04
- added J6: Barrel_Jack, symbol Connector:Barrel_Jack
- added Q5: 2SK4017(Q), symbol Simulation_SPICE:NMOS
- added R11, R13, R15, R26, R31: 180, symbol Device:R
- added R12, R14, R16, R17, R18, R19, R20: 1k, symbol Device:R
- added R21, R22, R27, R32: 100, symbol Device:R
- added R23, R24, R25, R28, R29, R30: 22k, symbol Device:R
- added RV1, RV2, RV3: 1k, symbol Device:R_Potentiometer
- added RV4, RV5, RV6: 1k, symbol Device:R_Potentiometer_Trim
- added U10: TBD62783A, symbol Transistor_Array:TBD62783A
- added U11, U14, U6: ${SIM.PARAMS}, symbol Simulation_SPICE:OPAMP
- added U2: 74AHC1G04, symbol 74xGxx:74AHC1G04
- added U3, U4, U5: PC817, Package_DIP:DIP-4_W7.62mm, symbol Isolator:PC817
- added U7: 74HC14, symbol 74xx:74HC14
- added U8: 74AHC04, symbol 74xx:74AHC04
- added U9: LM339, symbol Comparator:LM339
- R1: value R -> 180
- R2, R3, R5, R7: value R -> 50
- R4, R6, R8: value R -> 22k
Connections:
- net +3V3: now also U10.9 (VCC)
- net +5V: now also U1.4, C2.1, D1.2 (A), F1.1, J3.1 (Pin_1), J3.2 (Pin_2), J6.1, J7.1 (Pin_1), J7.2 (Pin_2), J9.1 (Pin_1), J9.2 (Pin_2), Q5.1 (D), RV1.1, RV2.1, RV3.1, U11.3 (V+), U14.3 (V+), U2.3 (GND), U3.4, U4.4, U5.4, U6.3 (V+), U7.14 (VCC), U8.14 (VCC), U9.3 (V+)
- net GND: now also A1.13 (GND), A1.18 (GND), A1.23 (GND), A1.28 (GND), A1.3 (GND), A1.38 (GND), A1.8 (GND), R1.2, C2.2, J6.2, R12.2, R14.2, R16.2, R17.2, R18.2, R19.2, R20.2, R24.2, R26.2, R29.2, R31.2, R32.2, RV1.3, RV2.3, RV3.3, U10.10 (GND), U10.11 (O8), U10.12 (O7), U10.13 (O6), U10.15 (O4), U10.17 (O2), U10.2 (I2), U10.4 (I4), U10.6 (I6), U10.7 (I7), U10.8 (I8), U11.4 (V-), U14.4 (V-), U2.5 (VCC), U6.4 (V-), U7.7 (GND), U8.7 (GND), U9.12 (V-); no longer R8.2
- net MOTOR_INPUT_1: now also U1.3
- net MOTOR_INPUT_2: now also U3.3
- net MOTOR_INPUT_3: now also U4.3
- net MOTOR_INPUT_4: now also U5.3
- net OPTO_INPUT_1: now also A1.14 (GPIO10)
- net at Q2.1 (D): now also Q1.1 (D), F1.2
- net at Q2.2 (G), R5.2: now also R19.1; no longer R6.1
- net at J2.2 (Pin_2), Q2.3 (S), Q4.1 (D): no longer R6.2
- net at Q4.2 (G), R7.2: now also R20.1; no longer R8.1
- net at Q3.2 (G), R3.2: now also R18.1; no longer R4.1
- net at Q1.2 (G), R2.2: now also R17.1; no longer R1.1
- net at J2.1 (Pin_1), Q1.3 (S), Q3.1 (D): no longer R1.2
- net OPTO_INPUT_2: now reaches A1.15 (GPIO11)
- net OPTO_INPUT_2: now also R11.1, U3.1
- net OPTO_INPUT_3: now reaches A1.16 (GPIO12)
- net OPTO_INPUT_3: now also R13.1, U4.1
- net OPTO_INPUT_4: now reaches A1.17 (GPIO13)
- net OPTO_INPUT_4: now also R15.1, U5.1
- net P_INPUT: now reaches A1.31 (GPIO26_ADC0)
- net P_INPUT: now also RV4.2
- net I_INPUT: now reaches A1.32 (GPIO27_ADC1)
- net I_INPUT: now also RV5.2
- net GNDA: now reaches A1.33 (AGND)
- net GNDA: now also RV4.3, RV5.3, RV6.3
- net D_INPUT: now reaches A1.34 (GPIO28_ADC2)
- net D_INPUT: now also RV6.2
- net +3.3VA: now reaches A1.35 (ADC_VREF)
- net +3.3VA: now also RV4.1, RV5.1, RV6.1
- net at A1.39 (VSYS): now also Q5.3 (S)
- net PHOTO_INTERUPTER_INPUT1: now reaches A1.4 (GPIO2)
- net PHOTO_INTERUPTER_INPUT1: now also U10.18 (O1)
- net at A1.40 (VBUS): now also U2.2
- net PHOTO_INTERUPTER_INPUT2: now reaches A1.5 (GPIO3)
- net PHOTO_INTERUPTER_INPUT2: now also U10.16 (O3)
- net PHOTO_INTERUPTER_INPUT3: now reaches A1.6 (GPIO4)
- net PHOTO_INTERUPTER_INPUT3: now also U10.14 (O5)
- new net: R11.2, R12.1, U3.2
- new net: Q5.2 (G), U2.4
- new net: R29.1, R30.1, U14.1 (+)
- new net: R28.2, U14.2 (-)
- new net: R27.2, U14.5
- new net: R13.2, R14.1, U4.2
- new net: U10.1 (I1), U9.2
- new net: J10.1 (Pin_1), U9.4 (-)
- new net: J10.2 (Pin_2), U9.5 (+)
- new net: R21.1, U7.1
- new net: J4.2 (Pin_2), U7.2, U8.1
- new net: D1.1 (K), R32.1
- new net: J7.3 (Pin_3), R25.2
- new net: J7.4 (Pin_4), R26.1
- new net: J11.1 (Pin_1), U9.6 (-)
- new net: J11.2 (Pin_2), U9.7 (+)
- new net: R24.1, R25.1, U11.1 (+)
- new net: R23.2, U11.2 (-)
- new net: R22.2, U11.5
- new net: J5.1 (Pin_1), U8.4
- new net: J5.2 (Pin_2), U7.4, U8.3
- new net: R27.1, U7.5
- new net: J8.2 (Pin_2), U7.6, U8.5
- new net: J4.1 (Pin_1), U8.2
- new net: R4.1, R6.1, U6.1 (+)
- new net: J3.3 (Pin_3), R6.2
- new net: R22.1, U7.3
- new net: J9.3 (Pin_3), R30.2
- new net: J9.4 (Pin_4), R31.1
- new net: U10.3 (I3), U9.1
- new net: J3.4 (Pin_4), R1.1
- new net: R28.1, RV3.2
- new net: R15.2, R16.1, U5.2
- new net: J8.1 (Pin_1), U8.6
- new net: R8.1, RV1.2
- new net: R8.2, U6.2 (-)
- new net: J12.1 (Pin_1), U9.10 (-)
- new net: J12.2 (Pin_2), U9.11 (+)
- new net: R21.2, U6.5
- new net: R23.1, RV2.2
- new net: U10.5 (I5), U9.13
Other:
- note added: "PHOTO INTERRUPTER SIGNAL 1...Anode, 2...Collector 3...Emitter 4...Cathode"
- moved on the sheet: A1, C1, J1, J2, M1, Q1, Q2, Q3, Q4, R10, R2, R3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
